File: wuerfel.kicad_sch (KiCad schematic)
At the start: 26 parts, among them IC1 M74HC4060YRM13TR, J1 PINHD_1x2_Female, Q1 BC857, SW1 SW_Push

Commit message: cleanup add folder pics
Parts:
- IC1: footprint SamacSys_Parts:SOIC127P600X175-16N -> Package_SO:SOIC-16_3.9x9.9mm_P1.27mm
Connections:
- no-connect marks 8 -> 7
Other:
- moved on the sheet: C2, D14, R3, R4, R5
Changed lines of the file:
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@@
 	)
 	(no_connect
-		(at 115.57 46.99)
-	)
-	(no_connect
 		(at 100.33 76.2)
 	)
@@
 	(wire
 		(pts
-			(xy 164.465 62.23) (xy 164.465 88.9)
+			(xy 165.1 62.23) (xy 165.1 88.9)
 		)
 		(stroke
@@
 	(wire
 		(pts
-			(xy 128.905 91.44) (xy 132.08 91.44)
+			(xy 129.54 91.44) (xy 132.08 91.44)
 		)
 		(stroke
@@
 	(wire
 		(pts
-			(xy 186.69 69.85) (xy 147.955 69.85)
+			(xy 186.69 69.85) (xy 148.59 69.85)
 		)
 		(stroke
@@
 	(wire
 		(pts
-			(xy 135.89 69.85) (xy 140.335 69.85)
+			(xy 135.89 69.85) (xy 140.97 69.85)
 		)
 		(stroke
@@
 	(wire
 		(pts
-			(xy 185.42 62.23) (xy 164.465 62.23)
+			(xy 185.42 62.23) (xy 165.1 62.23)
 		)
 		(stroke
@@
 	(wire
 		(pts
-			(xy 132.08 88.9) (xy 121.285 88.9)
+			(xy 132.08 88.9) (xy 121.92 88.9)
 		)
 		(stroke
@@
 	(wire
 		(pts
-			(xy 154.94 66.675) (xy 179.07 66.675)
+			(xy 154.94 67.31) (xy 179.07 67.31)
 		)
 		(stroke
@@
 	(wire
 		(pts
-			(xy 179.07 88.265) (xy 186.69 88.265)
+			(xy 179.07 88.9) (xy 186.69 88.9)
 		)
 		(stroke
@@
 	(wire
 		(pts
-			(xy 100.33 91.44) (xy 121.285 91.44)
+			(xy 100.33 91.44) (xy 121.92 91.44)
 		)
 		(stroke
@@
 	(wire
 		(pts
-			(xy 154.94 58.42) (xy 154.94 66.675)
+			(xy 154.94 58.42) (xy 154.94 67.31)
 		)
 		(stroke
@@
 	(wire
 		(pts
-			(xy 121.285 86.36) (xy 111.76 86.36)
+			(xy 121.92 86.36) (xy 111.76 86.36)
 		)
 		(stroke
@@
 	(wire
 		(pts
-			(xy 186.69 88.265) (xy 186.69 100.33)
+			(xy 186.69 88.9) (xy 186.69 100.33)
 		)
 		(stroke
@@
 	(wire
 		(pts
-			(xy 51.435 134.62) (xy 45.72 134.62)
+			(xy 52.07 134.62) (xy 45.72 134.62)
 		)
 		(stroke
@@
 	(wire
 		(pts
-			(xy 59.055 134.62) (xy 62.23 134.62)
+			(xy 59.69 134.62) (xy 62.23 134.62)
 		)
 		(stroke
@@
 	(wire
 		(pts
-			(xy 100.33 88.9) (xy 113.665 88.9)
+			(xy 100.33 88.9) (xy 114.3 88.9)
 		)
 		(stroke
@@
 	(wire
 		(pts
-			(xy 179.07 66.675) (xy 179.07 88.265)
+			(xy 179.07 67.31) (xy 179.07 88.9)
 		)
 		(stroke
@@
 	(wire
 		(pts
-			(xy 128.905 86.36) (xy 132.08 86.36)
+			(xy 129.54 86.36) (xy 132.08 86.36)
 		)
 		(stroke
@@
 	(wire
 		(pts
-			(xy 154.94 88.9) (xy 164.465 88.9)
+			(xy 154.94 88.9) (xy 165.1 88.9)
 		)
 		(stroke
@@
 	(symbol
 		(lib_id "Device:R")
-		(at 144.145 69.85 90)
+		(at 144.78 69.85 90)
 		(unit 1)
 		(exclude_from_sim no)
@@
 		(fields_autoplaced yes)
 		(property "Reference" "R5"
-			(at 144.145 63.5 90)
+			(at 144.78 63.5 90)
 			(effects
 				(font
@@
 		)
 		(property "Value" "390R"
-			(at 144.145 66.04 90)
+			(at 144.78 66.04 90)
 			(effects
 				(font
@@
 		)
 		(property "Footprint" "Resistor_SMD:R_1206_3216Metric_Pad1.30x1.75mm_HandSolder"
-			(at 144.145 71.628 90)
+			(at 144.78 71.628 90)
 			(effects
 				(font
@@
 		)
 		(property "Datasheet" "~"
-			(at 144.145 69.85 0)
+			(at 144.78 69.85 0)
 			(effects
 				(font
@@
 		)
 		(property "Description" ""
-			(at 144.145 69.85 0)
+			(at 144.78 69.85 0)
 			(effects
 				(font
@@
 	(symbol
 		(lib_id "Device:R")
-		(at 117.475 88.9 90)
+		(at 118.11 88.9 90)
 		(unit 1)
 		(exclude_from_sim no)
@@
 		(fields_autoplaced yes)
 		(property "Reference" "R3"
-			(at 117.475 82.55 90)
+			(at 118.11 82.55 90)
 			(effects
 				(font
@@
 		)
 		(property "Value" "220k"
-			(at 117.475 85.09 90)
+			(at 118.11 85.09 90)
 			(effects
 				(font
@@
 		)
 		(property "Footprint" "Resistor_SMD:R_1206_3216Metric_Pad1.30x1.75mm_HandSolder"
-			(at 117.475 90.678 90)
+			(at 118.11 90.678 90)
 			(effects
 				(font
@@
 		)
 		(property "Datasheet" "~"
-			(at 117.475 88.9 0)
+			(at 118.11 88.9 0)
 			(effects
 				(font
@@
 		)
 		(property "Description" ""
-			(at 117.475 88.9 0)
+			(at 118.11 88.9 0)
 			(effects
 				(font
@@
 	(symbol
 		(lib_id "Device:C")
-		(at 125.095 91.44 90)
+		(at 125.73 91.44 90)
 		(unit 1)
 		(exclude_from_sim no)
@@
 		(dnp no)
 		(property "Reference" "C2"
-			(at 125.095 95.25 90)
+			(at 125.73 95.25 90)
 			(effects
 				(font
@@
 		)
 		(property "Value" "220p"
-			(at 125.095 97.79 90)
+			(at 125.73 97.79 90)
 			(effects
 				(font
@@
 		)
 		(property "Footprint" "Capacitor_SMD:C_0805_2012Metric_Pad1.18x1.45mm_HandSolder"
-			(at 128.905 90.4748 0)
+			(at 129.54 90.4748 0)
 			(effects
 				(font
@@
 		)
 		(property "Datasheet" "~"
-			(at 125.095 91.44 0)
+			(at 125.73 91.44 0)
 			(effects
 				(font
@@
 		)
 		(property "Description" ""
-			(at 125.095 91.44 0)
+			(at 125.73 91.44 0)
 			(effects
 				(font
@@
 	(symbol
 		(lib_id "Device:R")
-		(at 125.095 86.36 90)
+		(at 125.73 86.36 90)
 		(unit 1)
 		(exclude_from_sim no)
@@
 		(fields_autoplaced yes)
 		(property "Reference" "R4"
-			(at 125.095 80.01 90)
+			(at 125.73 80.01 90)
 			(effects
 				(font
@@
 		)
 		(property "Value" "470k"
-			(at 125.095 82.55 90)
+			(at 125.73 82.55 90)
 			(effects
 				(font
@@
 		)
 		(property "Footprint" "Resistor_SMD:R_1206_3216Metric_Pad1.30x1.75mm_HandSolder"
-			(at 125.095 88.138 90)
+			(at 125.73 88.138 90)
 			(effects
 				(font
@@
 		)
 		(property "Datasheet" "~"
-			(at 125.095 86.36 0)
+			(at 125.73 86.36 0)
 			(effects
 				(font
@@
 		)
 		(property "Description" ""
-			(at 125.095 86.36 0)
+			(at 125.73 86.36 0)
 			(effects
 				(font
@@
 			)
 		)
-		(property "Footprint" "SamacSys_Parts:SOIC127P600X175-16N"
+		(property "Footprint" "Package_SO:SOIC-16_3.9x9.9mm_P1.27mm"
 			(at 96.52 168.58 0)
 			(effects
@@
 	(symbol
 		(lib_id "Diode:LL4148")
-		(at 55.245 134.62 180)
+		(at 55.88 134.62 180)
 		(unit 1)
 		(exclude_from_sim no)
@@
 		(fields_autoplaced yes)
 		(property "Reference" "D14"
-			(at 55.245 128.27 0)
+			(at 55.88 128.27 0)
 			(effects
 				(font
@@
 		)
 		(property "Value" "LL4148"
-			(at 55.245 130.81 0)
+			(at 55.88 130.81 0)
 			(effects
 				(font
@@
 		)
 		(property "Footprint" "Diode_SMD:D_MiniMELF"
-			(at 55.245 130.175 0)
+			(at 55.88 130.175 0)
 			(effects
 				(font
@@
 		)
 		(property "Datasheet" "http://www.vishay.com/docs/85557/ll4148.pdf"
-			(at 55.245 134.62 0)
+			(at 55.88 134.62 0)
 			(effects
 				(font
@@
 		)
 		(property "Description" ""
-			(at 55.245 134.62 0)
+			(at 55.88 134.62 0)
 			(effects
 				(font
@@
 		)
 		(property "Sim.Device" "D"
-			(at 55.245 134.62 0)
+			(at 55.88 134.62 0)
 			(effects
 				(font
@@
 		)
 		(property "Sim.Pins" "1=K 2=A"
-			(at 55.245 134.62 0)
+			(at 55.88 134.62 0)
 			(effects
 				(font
